Commit message: add realsense camera from realsense_description package

File: niagara_model/urdf/zed2.xacro (robot description, xacro)
@@ -10,4 +10,8 @@
         <origin xyz="0.17 0 0.07" rpy="0 0 0"/>
     </joint>
+    <xacro:include filename="$(find realsense2_description)/urdf/_d455.urdf.xacro" />
+    <xacro:sensor_d455 parent="zed_camera_link" name="D455" use_nominal_extrinsics="true">
+      <origin xyz="0 0 0" rpy="0 0 0"/>
+    </xacro:sensor_d455>
     <link name="zed_camera_link">
       <inertial>
@@ -19,5 +23,5 @@
         <origin xyz="0 0 0" rpy="0 0 0"/>
         <geometry>
-          <box size="0.02 0.1 0.02"/>
+          <box size="0.01 0.08 0.02"/>
         </geometry>
       </collision>
@@ -25,5 +29,5 @@
         <origin xyz="0 0 0" rpy="0 0 0"/>
         <geometry>
-          <box size="0.02 0.1 0.02"/>
+          <box size="0.01 0.08 0.02"/>
         </geometry>
         <material name="red"/>
