Commit message: change urdfs to match bearcar

File: niagara_model/urdf/Autoreifen.xacro (robot description, xacro)
@@ -1,27 +1,27 @@
 <?xml version="1.0"?>
 <robot name="dasautonomeauto" xmlns:xacro="http://www.ros.org/wiki/xacro">
-  <xacro:property name="tire_dia" value="0.350"/>  <!-- Reduced from 0.440 -->
-  <xacro:property name="tire_width" value="0.195"/>  <!-- Reduced from 0.195 -->
-  <xacro:property name="hub_dia" value="0.235"/>  <!-- Reduced from 0.235 -->
-  <xacro:property name="hex_hub_depth" value="0.120"/> <!-- or +0.072 -->
-  <xacro:property name="wheel_mass" value="8.0"/>   <!-- check -->
-  <xacro:property name="wheelbase" value="2.1"/>
-  <xacro:property name="hex_hub_dist" value="0.9191"/>
-  <xacro:property name="wheel_travel" value="0.209492959255614"/>
-  <xacro:property name="axle_eff_limit" value="204.95"/>
-  <xacro:property name="axle_vel_limit" value="39.02"/>
+  <xacro:property name="tire_dia" value="0.07"/>  <!-- Reduced from 0.440 OLD = 0.350-->
+  <xacro:property name="tire_width" value="0.02"/>  <!-- Reduced from 0.195 OLD: 0.195-->
+  <xacro:property name="hub_dia" value="0.001"/>  <!-- Reduced from 0.235 OLD: 0.235 -->
+  <xacro:property name="hex_hub_depth" value="0.008"/> <!-- or +0.072 OLD: 120-->
+  <xacro:property name="wheel_mass" value="0.1"/>   <!-- check  OLD: 8.0-->
+  <xacro:property name="wheelbase" value="0.206"/>
+  <xacro:property name="hex_hub_dist" value="0.005"/>
+  <xacro:property name="wheel_travel" value="0.0209492959255614"/>
+  <xacro:property name="axle_eff_limit" value="20.495"/>
+  <xacro:property name="axle_vel_limit" value="3.902"/>
   <!-- Properties of the car -->
-  <xacro:property name="front_wheel_x" value="0.787346576344423"/>
-  <xacro:property name="front_wheel_y" value="0.495625727164768"/>
-  <xacro:property name="front_wheel_z" value="0.1094929592556163"/>
-  <xacro:property name="rear_wheel_x" value="1.04780116842239"/>
-  <xacro:property name="rear_wheel_y" value="0.495625727164768"/>
-  <xacro:property name="rear_wheel_z" value="0.1094929592556163"/>
+  <xacro:property name="front_wheel_x" value="0.1"/>
+  <xacro:property name="front_wheel_y" value="0.105"/>
+  <xacro:property name="front_wheel_z" value="0.1"/>
+  <xacro:property name="rear_wheel_x" value="0.1"/>
+  <xacro:property name="rear_wheel_y" value="-0.105"/>
+  <xacro:property name="rear_wheel_z" value="0.1"/>
   <!-- Degree-to-radian conversions -->
   <xacro:property name="degrees_45" value="0.785398163"/>
   <xacro:property name="degrees_90" value="1.57079633"/>
   <xacro:property name="degrees_180" value="3.14159265"/>
-  <xacro:property name="servo_stall_torque" value="50"/>  <!-- check -->
-  <xacro:property name="servo_no_load_speed" value="25"/> <!-- check -->
+  <xacro:property name="servo_stall_torque" value="5"/>  <!-- check -->
+  <xacro:property name="servo_no_load_speed" value="2.5"/> <!-- check -->
   <material name="black">
       <color rgba="0 0 0 1"/>

File: niagara_model/urdf/DasAutonomeAuto.urdf (robot description, URDF)
Before this commit: robot dasautonomeauto, 2 links, 1 joints
Links:
- link base_link: mass 125.0 -> 2.0; geometry collision box size=0.34 0.17 0.20; visual box size=0.34 0.17 0.20
Joints:
- joint base_footprint_joint: origin xyz=0 0 0.2 rpy=0 0 0 -> xyz=0 0 0 rpy=0 0 0

File: niagara_model/urdf/VLP-16.xacro (robot description, xacro)
@@ -2,7 +2,7 @@
 <robot xmlns:xacro="http://www.ros.org/wiki/xacro" name="VLP-16">
   <xacro:property name="M_PI" value="3.1415926535897931"/>
-  <xacro:macro name="VLP-16" params="parent:=base_link name:=velodyne topic:=/velodyne_points hz:=10 lasers:=16 samples:=1875 collision_range:=0.3 min_range:=0.9 max_range:=130.0 noise:=0.008 min_angle:=-${M_PI} max_angle:=${M_PI} gpu:=false">
+  <xacro:macro name="VLP-16" params="parent:=base_link name:=velodyne topic:=/LaserScan hz:=10 lasers:=16 samples:=1875 collision_range:=0.3 min_range:=0.9 max_range:=130.0 noise:=0.008 min_angle:=-${M_PI} max_angle:=${M_PI} gpu:=false">
     <joint name="${name}_base_mount_joint" type="fixed">
-      <origin xyz="0 0 1" rpy="0 0 0" />
+      <origin xyz="0 0 0.1" rpy="0 0 0" />
       <parent link="${parent}"/>
       <child link="${name}_base_link"/>
@@ -11,5 +11,5 @@
       <inertial>
         <mass value="0.83"/>
-        <origin xyz="0 0 0.03585"/>
+        <origin xyz="0 0 0.0225"/>
         <inertia ixx="${(0.83 * (3.0*0.0516*0.0516 + 0.0717*0.0717)) / 12.0}" ixy="0" ixz="0" iyy="${(0.83 * (3.0*0.0516*0.0516 + 0.0717*0.0717)) / 12.0}" iyz="0" izz="${0.5 * 0.83 * (0.0516*0.0516)}"/>
       </inertial>

File: niagara_model/urdf/imu.xacro (robot description, xacro)
@@ -37,5 +37,5 @@
     <joint name="imu_joint" type="fixed">
         <parent link="base_link"/>
-        <child link="imu_link"/>
+        <child link="imu_link"/>Topic
         <origin xyz="0 0 0.01"/>
     </joint>

Commit message: change urdf to match bearcar, adjust initial position

File: niagara_model/urdf/Autoreifen.xacro (robot description, xacro)
@@ -1,11 +1,20 @@
 <?xml version="1.0"?>
 <robot name="dasautonomeauto" xmlns:xacro="http://www.ros.org/wiki/xacro">
-  <xacro:property name="tire_dia" value="0.07"/>  <!-- Reduced from 0.440 OLD = 0.350-->
-  <xacro:property name="tire_width" value="0.02"/>  <!-- Reduced from 0.195 OLD: 0.195-->
-  <xacro:property name="hub_dia" value="0.001"/>  <!-- Reduced from 0.235 OLD: 0.235 -->
-  <xacro:property name="hex_hub_depth" value="0.008"/> <!-- or +0.072 OLD: 120-->
+  <xacro:property name="tire_dia" value="0.12"/>  <!-- Reduced from 0.440 OLD = 0.350-->
+  <xacro:property name="tire_width" value="0.06"/>  <!-- Reduced from 0.195 OLD: 0.195-->
+  <xacro:property name="hub_dia" value="0.00"/>  <!-- Reduced from 0.235 OLD: 0.235 -->
+  <!-- hub_dia and tire_dia are the diameters of the hub and tire,
+       respectively. hex_hub_depth is the distance that the hex hub is
+       inset from the outer edge of the tire. It is set so that each wheel
+       is a "zero offset" wheel. hex_hub_depth = tire_width / 2 -
+       axle_length. -->
+  <xacro:property name="hex_hub_depth" value="0.0319"/> <!-- or +0.072 OLD: 120-->
   <xacro:property name="wheel_mass" value="0.1"/>   <!-- check  OLD: 8.0-->
-  <xacro:property name="wheelbase" value="0.206"/>
-  <xacro:property name="hex_hub_dist" value="0.005"/>
+  <!-- hex_hub_dist is the distance between left and right hex hubs when
+       the shock absorbers are fully extended. axle_length is the distance
+       from a U joint to the corresponding hex hub. wheel_travel is the
+       vertical wheel travel. -->
+  <xacro:property name="wheelbase" value="024"/>
+  <xacro:property name="hex_hub_dist" value="0.18"/>
   <xacro:property name="wheel_travel" value="0.0209492959255614"/>
   <xacro:property name="axle_eff_limit" value="20.495"/>
@@ -22,5 +31,5 @@
   <xacro:property name="degrees_90" value="1.57079633"/>
   <xacro:property name="degrees_180" value="3.14159265"/>
-  <xacro:property name="servo_stall_torque" value="5"/>  <!-- check -->
+  <xacro:property name="servo_stall_torque" value="3"/>  <!-- check -->
   <xacro:property name="servo_no_load_speed" value="2.5"/> <!-- check -->
   <material name="black">
@@ -43,5 +52,5 @@
   <xacro:macro name="null_inertial">
     <inertial>
-      <mass value="4.5"/>
+      <mass value="0.5"/>
       <inertia ixx="0.001" ixy="0" ixz="0" iyy="0.001" iyz="0" izz="0.001"/>
     </inertial>

File: niagara_model/urdf/DasAutonomeAuto.urdf (robot description, URDF)
Before this commit: robot dasautonomeauto, 2 links, 1 joints
Links:
- link base_link: mass 2.0 -> 1.0

File: niagara_model/urdf/zed2.xacro (robot description, xacro)
@@ -8,16 +8,16 @@
         <parent link="base_link"/>
         <child link="zed_camera_link"/>
-        <origin xyz="0.6 0 0.6" rpy="0 0 0"/>
+        <origin xyz="0.17 0 0.07" rpy="0 0 0"/>
     </joint>
     <link name="zed_camera_link">
       <inertial>
-        <mass value="1e-5" />
+        <mass value="0.0" />
         <origin xyz="0 0 0" rpy="0 0 0"/>
-        <inertia ixx="1e-6" ixy="0" ixz="0" iyy="1e-6" iyz="0" izz="1e-6" />
+        <inertia ixx="0" ixy="0" ixz="0" iyy="0" iyz="0" izz="0" />
       </inertial>
       <collision>
         <origin xyz="0 0 0" rpy="0 0 0"/>
         <geometry>
-          <box size="0.033 0.175 0.030"/>
+          <box size="0.02 0.1 0.02"/>
         </geometry>
       </collision>
@@ -25,5 +25,5 @@
         <origin xyz="0 0 0" rpy="0 0 0"/>
         <geometry>
-          <box size="0.033 0.175 0.030"/>
+          <box size="0.02 0.1 0.02"/>
         </geometry>
         <material name="red"/>

Commit message: delete waypoint packages, fix wheel positions

File: niagara_model/urdf/Autoreifen.xacro (robot description, xacro)
@@ -22,8 +22,8 @@
   <!-- Properties of the car -->
   <xacro:property name="front_wheel_x" value="0.1"/>
-  <xacro:property name="front_wheel_y" value="0.105"/>
+  <xacro:property name="front_wheel_y" value="0.125"/>
   <xacro:property name="front_wheel_z" value="0.1"/>
   <xacro:property name="rear_wheel_x" value="0.1"/>
-  <xacro:property name="rear_wheel_y" value="-0.105"/>
+  <xacro:property name="rear_wheel_y" value="-0.125"/>
   <xacro:property name="rear_wheel_z" value="0.1"/>
   <!-- Degree-to-radian conversions -->

Commit message: remove waypoint stuff, fix movement when starting simulation

File: niagara_model/urdf/Autoreifen.xacro (robot description, xacro)
@@ -10,5 +10,5 @@
        axle_length. -->
   <xacro:property name="hex_hub_depth" value="0.0319"/> <!-- or +0.072 OLD: 120-->
-  <xacro:property name="wheel_mass" value="0.1"/>   <!-- check  OLD: 8.0-->
+  <xacro:property name="wheel_mass" value="0.2"/>   <!-- check  OLD: 8.0-->
   <!-- hex_hub_dist is the distance between left and right hex hubs when
        the shock absorbers are fully extended. axle_length is the distance
@@ -100,4 +100,5 @@
       <axis xyz="0 0 -1"/>
       <limit effort="${axle_eff_limit}" velocity="${axle_vel_limit}"/>
+      <dynamics damping="0.05" friction="0.1"/>
     </joint>
     <gazebo reference="${lr_prefix}_${fr_prefix}_wheel">
@@ -135,4 +136,5 @@
       <axis xyz="0 0 -1"/>
       <limit effort="${axle_eff_limit}" velocity="${axle_vel_limit}"/>
+      <dynamics damping="0.05" friction="0.1"/>
     </joint>
     <gazebo reference="${lr_prefix}_${fr_prefix}_wheel">

File: niagara_model/urdf/DasAutonomeAuto.urdf (robot description, URDF)
Before this commit: robot dasautonomeauto, 2 links, 1 joints
Links:
- link base_link: mass 1.0 -> 50.0
