Commit message: fix typo

File: niagara_model/urdf/imu.xacro (robot description, xacro)
@@ -37,5 +37,5 @@
     <joint name="imu_joint" type="fixed">
         <parent link="base_link"/>
-        <child link="imu_link"/>Topic
+        <child link="imu_link"/>
         <origin xyz="0 0 0.01"/>
     </joint>
